File: UART.sch (KiCad schematic (older format))
At the start: 7 parts, among them U4 8250, U5 FTDI-USB

Commit message: RevB
Parts:
- removed RN3: 10K, Resistor_THT:R_Array_SIP6, symbol Device:R_Network05_US
- removed U5: FTDI-USB, 8085:FTDI_USB, symbol 8085:FTDI-USB
- added C11: 10nF, Capacitor_SMD:C_0805_2012Metric_Pad1.15x1.40mm_HandSolder, symbol Device:C
- added C12, C13, C15: 0.1uF, Capacitor_SMD:C_0805_2012Metric_Pad1.15x1.40mm_HandSolder, symbol Device:C
- added C14: 1uF, Capacitor_THT:CP_Radial_D5.0mm_P2.50mm, symbol Device:CP1
- added D2: POWER, LED_SMD:LED_0805_2012Metric_Pad1.15x1.40mm_HandSolder, symbol Device:LED_Small
- added D3: TX, LED_SMD:LED_0805_2012Metric_Pad1.15x1.40mm_HandSolder, symbol Device:LED_Small
- added D4: RX, LED_SMD:LED_0805_2012Metric_Pad1.15x1.40mm_HandSolder, symbol Device:LED_Small
- added J1: USB_B, 8085:USB_B_OST_USB-B1HSxx_Horizontal, symbol Connector:USB_B
- added L1: MI0805K400R-10, Inductor_SMD:L_0805_2012Metric_Pad1.15x1.40mm_HandSolder, symbol Device:Ferrite_Bead_Small
- added Q2: IRLML6402, Package_TO_SOT_SMD:SOT-23, symbol Transistor_FET:IRLML6402
- added R4: 10K, Resistor_SMD:R_0805_2012Metric_Pad1.15x1.40mm_HandSolder, symbol Device:R
- added R5: 1K, Resistor_SMD:R_0805_2012Metric_Pad1.15x1.40mm_HandSolder, symbol Device:R
- added RN3: 10K, Resistor_SMD:R_Array_Convex_4x1206, symbol Device:R_Pack04
- added RN5: 330, Resistor_SMD:R_Array_Convex_4x1206, symbol Device:R_Pack04
- added U5: FT232RL, Package_SO:SSOP-28_5.3x10.2mm_P0.65mm, symbol Interface_USB:FT232RL
Connections:
- net labels added: D+, D-, TXDEN, VBUS, VIN, ~PWREN, ~RXLED, ~SLEEP, ~TXLED
- wire segments 61 -> 122
- no-connect marks 9 -> 10
Other:
- moved on the sheet: JP1, JP2, JP3, JP4
