File: CPU.sch (KiCad schematic (older format))
At the start: 10 parts, among them SW1 RESET, U7 8085, U8 74LS573, Y1 4MHz

Commit message: RevB
Parts:
- removed RN1: 10K, Resistor_THT:R_Array_SIP8, symbol Device:R_Network07_US
- removed RN2: 10K, Resistor_THT:R_Array_SIP6, symbol Device:R_Network05_US
- added RN1, RN2, RN4: 10K, Resistor_SMD:R_Array_Convex_4x1206, symbol Device:R_Pack04
- D1: footprint Diode_THT:D_DO-35_SOD27_P10.16mm_Horizontal -> Diode_SMD:D_MiniMELF
Connections:
- net labels added: READY
- wire segments 93 -> 103
Changed lines of the file:
@@
 EESchema Schematic File Version 4
-LIBS:CPU8085-cache
-EELAYER 26 0
+EELAYER 30 0
 EELAYER END
 $Descr USLetter 11000 8500
@@
 F 0 "D1" V 1450 3200 50  0000 L CNN
 F 1 "1N4004" V 1495 3429 50  0001 L CNN
-F 2 "Diode_THT:D_DO-35_SOD27_P10.16mm_Horizontal" H 1450 3350 50  0001 C CNN
+F 2 "Diode_SMD:D_MiniMELF" H 1450 3350 50  0001 C CNN
 F 3 "~" H 1450 3350 50  0001 C CNN
 	1    1450 3350
@@
 Wire Wire Line
 	3400 2700 3500 2700
-$Comp
-L Device:R_Network07_US RN1
-U 1 1 5B9E4051
-P 2400 1500
-F 0 "RN1" H 2020 1454 50  0000 R CNN
-F 1 "10K" H 2020 1545 50  0000 R CNN
-F 2 "Resistor_THT:R_Array_SIP8" V 2875 1500 50  0001 C CNN
-F 3 "http://www.vishay.com/docs/31509/csc.pdf" H 2400 1500 50  0001 C CNN
-	1    2400 1500
-	-1   0    0    1
-$EndComp
 Wire Wire Line
 	3350 2700 3350 2500
 Wire Wire Line
 	3350 2500 3500 2500
-$Comp
-L Device:R_Network05_US RN2
-U 1 1 5BA06FF5
-P 3250 1500
-F 0 "RN2" H 2970 1546 50  0000 R CNN
-F 1 "10K" H 2970 1455 50  0000 R CNN
-F 2 "Resistor_THT:R_Array_SIP6" V 3625 1500 50  0001 C CNN
-F 3 "http://www.vishay.com/docs/31509/csc.pdf" H 3250 1500 50  0001 C CNN
-	1    3250 1500
-	-1   0    0    -1
-$EndComp
 Text Label 5300 4400 0    50   ~ 0
 ~RD
@@
 L power:VCC #PWR020
 U 1 1 5BA1BE66
-P 3450 1300
-F 0 "#PWR020" H 3450 1150 50  0001 C CNN
-F 1 "VCC" H 3467 1473 50  0000 C CNN
-F 2 "" H 3450 1300 50  0001 C CNN
-F 3 "" H 3450 1300 50  0001 C CNN
-	1    3450 1300
-	1    0    0    -1
-$EndComp
-Wire Wire Line
-	3350 2100 3500 2100
+P 3350 1300
+F 0 "#PWR020" H 3350 1150 50  0001 C CNN
+F 1 "VCC" H 3367 1473 50  0000 C CNN
+F 2 "" H 3350 1300 50  0001 C CNN
+F 3 "" H 3350 1300 50  0001 C CNN
+	1    3350 1300
+	1    0    0    -1
+$EndComp
 Wire Wire Line
 	3150 1700 3150 2000
 Wire Wire Line
-	3050 1700 3050 2000
-Wire Wire Line
-	3350 1700 3350 2100
-Wire Wire Line
-	3250 1700 3250 2000
+	3350 1700 3350 2000
 Text Label 5300 4200 0    50   ~ 0
 IO~M
+Text Label 3150 1900 1    50   ~ 0
+IO~M
 Text Label 3250 1850 1    50   ~ 0
-IO~M
-Text Label 3150 1850 1    50   ~ 0
 ~RD
-Text Label 3050 1850 1    50   ~ 0
+Text Label 3350 1850 1    50   ~ 0
 ~WR
 $Comp
@@
 Wire Wire Line
 	4900 5300 5150 5300
-Wire Wire Line
-	3450 1700 3750 1700
-Wire Wire Line
-	3750 1700 3750 1300
-Wire Wire Line
-	3750 1300 3450 1300
-Connection ~ 3450 1300
 Wire Wire Line
 	2700 1300 2700 1000
@@
 Text HLabel 2250 3100 0    50   Input ~ 0
 TRAP
-Text Label 2700 1300 1    50   ~ 0
+Text Label 2100 1300 1    50   ~ 0
 HOLD
-Text Label 2600 1300 1    50   ~ 0
+Text Label 2200 1250 1    50   ~ 0
 SID
-Text Label 2500 1300 1    50   ~ 0
+Text Label 2300 1300 1    50   ~ 0
 TRAP
 Text Label 2400 1300 1    50   ~ 0
 RST7_5
-Text Label 2300 1300 1    50   ~ 0
+Text Label 2500 1300 1    50   ~ 0
 RST6_5
-Text Label 2200 1300 1    50   ~ 0
+Text Label 2600 1300 1    50   ~ 0
 RST5_5
-Text Label 2100 1300 1    50   ~ 0
+Text Label 2700 1250 1    50   ~ 0
 INTR
 Wire Wire Line
@@
 	9600 1500 9600 1300
 Connection ~ 9600 1500
+$Comp
+L Device:R_Pack04 RN1
+U 1 1 5BA35285
+P 2200 1500
+F 0 "RN1" H 1750 1550 50  0000 L CNN
+F 1 "10K" H 1750 1450 50  0000 L CNN
+F 2 "Resistor_SMD:R_Array_Convex_4x1206" V 2475 1500 50  0001 C CNN
+F 3 "~" H 2200 1500 50  0001 C CNN
+	1    2200 1500
+	1    0    0    -1
+$EndComp
+$Comp
+L Device:R_Pack04 RN2
+U 1 1 5BA352E9
+P 2600 1500
+F 0 "RN2" H 2800 1550 50  0000 L CNN
+F 1 "10K" H 2800 1450 50  0000 L CNN
+F 2 "Resistor_SMD:R_Array_Convex_4x1206" V 2875 1500 50  0001 C CNN
+F 3 "~" H 2600 1500 50  0001 C CNN
+	1    2600 1500
+	1    0    0    -1
+$EndComp
+$Comp
+L Device:R_Pack04 RN4
+U 1 1 5BA3533F
+P 3250 1500
+F 0 "RN4" H 3438 1546 50  0000 L CNN
+F 1 "10K" H 3438 1455 50  0000 L CNN
+F 2 "Resistor_SMD:R_Array_Convex_4x1206" V 3525 1500 50  0001 C CNN
+F 3 "~" H 3250 1500 50  0001 C CNN
+	1    3250 1500
+	1    0    0    -1
+$EndComp
+Wire Wire Line
+	3050 1300 3150 1300
+Connection ~ 3350 1300
+Connection ~ 3150 1300
+Wire Wire Line
+	3150 1300 3250 1300
+Connection ~ 3250 1300
+Wire Wire Line
+	3250 1300 3350 1300
+Wire Wire Line
+	2000 1700 2100 1700
+Wire Wire Line
+	2100 1700 2200 1700
+Connection ~ 2100 1700
+Wire Wire Line
+	2200 1700 2300 1700
+Connection ~ 2200 1700
+Wire Wire Line
+	2300 1700 2400 1700
+Connection ~ 2300 1700
+Wire Wire Line
+	2400 1700 2500 1700
+Connection ~ 2400 1700
+Wire Wire Line
+	2500 1700 2600 1700
+Connection ~ 2500 1700
+Wire Wire Line
+	2600 1700 2700 1700
+Connection ~ 2600 1700
+Connection ~ 2700 1700
+Wire Wire Line
+	2000 1300 1700 1300
+Wire Wire Line
+	1700 1300 1700 1700
+Wire Wire Line
+	1700 1700 2000 1700
+Connection ~ 2000 1700
+Wire Wire Line
+	3050 2100 3050 1700
+Text Label 3150 2100 0    50   ~ 0
+READY
+Wire Wire Line
+	3050 2100 3500 2100
+Wire Wire Line
+	3250 1700 3250 2000
+Wire Wire Line
+	4900 2800 6900 2800
+Wire Wire Line
+	4900 2700 6800 2700
+Wire Wire Line
+	4900 2600 6700 2600
+Wire Wire Line
+	4900 2500 6600 2500
+Wire Wire Line
+	4900 2400 6500 2400
+Wire Wire Line
+	4900 2300 6400 2300
+Wire Wire Line
+	4900 2200 6300 2200
+Wire Wire Line
+	4900 2100 6200 2100
 Wire Bus Line
 	5750 1250 5750 2700
-Wire Wire Line
-	4900 2800 6900 2800
-Wire Wire Line
-	4900 2700 6800 2700
-Wire Wire Line
-	4900 2600 6700 2600
-Wire Wire Line
-	4900 2500 6600 2500
-Wire Wire Line
-	4900 2400 6500 2400
-Wire Wire Line
-	4900 2300 6400 2300
-Wire Wire Line
-	4900 2200 6300 2200
-Wire Wire Line
-	4900 2100 6200 2100
+Wire Bus Line
+	8900 1300 8900 2250
 Wire Bus Line
 	9600 1500 9600 3500
-Wire Bus Line
-	8900 1300 8900 2250
 $EndSCHEMATC

Commit message: RevC
Parts:
- removed C8: 1uF, Capacitor_THT:CP_Radial_D5.0mm_P2.50mm, symbol Device:CP1
- removed D1: 1N4004, Diode_SMD:D_MiniMELF, symbol Device:D_ALT
- removed R1: 75K, Resistor_THT:R_Axial_DIN0207_L6.3mm_D2.5mm_P10.16mm_Horizontal, symbol Device:R_US
- added U5: MCP1319T-46LE, Package_TO_SOT_SMD:SOT-23-5_HandSoldering, symbol 8085:MCP1319
- SW1: footprint Connector_PinHeader_2.54mm:PinHeader_1x02_P2.54mm_Vertical -> 8085:Switch_Tactile_SMD_6x6mm_PTS645
Connections:
- wire segments 103 -> 101
- no-connect marks 5 -> 6
Other:
- moved on the sheet: SW1
Changed lines of the file:
@@
 Sheet 5 6
 Title "CPU"
-Date "2018-09-17"
-Rev "A"
+Date "2018-09-27"
+Rev "C"
 Comp ""
 Comment1 ""
@@
 Comment4 ""
 $EndDescr
-$Comp
-L Device:R_US R1
-U 1 1 5B8C097C
-P 950 3350
-F 0 "R1" H 1018 3396 50  0000 L CNN
-F 1 "75K" H 1018 3305 50  0000 L CNN
-F 2 "Resistor_THT:R_Axial_DIN0207_L6.3mm_D2.5mm_P10.16mm_Horizontal" V 990 3340 50  0001 C CNN
-F 3 "~" H 950 3350 50  0001 C CNN
-	1    950  3350
-	1    0    0    -1
-$EndComp
-$Comp
-L power:VCC #PWR016
-U 1 1 5B8C0DD8
-P 950 3200
-F 0 "#PWR016" H 950 3050 50  0001 C CNN
-F 1 "VCC" H 967 3373 50  0000 C CNN
-F 2 "" H 950 3200 50  0001 C CNN
-F 3 "" H 950 3200 50  0001 C CNN
-	1    950  3200
-	1    0    0    -1
-$EndComp
-$Comp
-L Device:D_ALT D1
-U 1 1 5B8C0E93
-P 1450 3350
-F 0 "D1" V 1450 3200 50  0000 L CNN
-F 1 "1N4004" V 1495 3429 50  0001 L CNN
-F 2 "Diode_SMD:D_MiniMELF" H 1450 3350 50  0001 C CNN
-F 3 "~" H 1450 3350 50  0001 C CNN
-	1    1450 3350
-	0    1    1    0
-$EndComp
-Connection ~ 950  3200
-Connection ~ 950  3500
 NoConn ~ 4900 4000
 NoConn ~ 4900 4100
-Wire Wire Line
-	4900 4900 6850 4900
-Wire Wire Line
-	950  3500 1450 3500
 NoConn ~ 4900 5100
 NoConn ~ 4900 4800
@@
 L Switch:SW_DIP_x01 SW1
 U 1 1 5B8C4B7C
-P 950 3800
-F 0 "SW1" V 996 3670 50  0000 R CNN
-F 1 "RESET" V 905 3670 50  0000 R CNN
-F 2 "Connector_PinHeader_2.54mm:PinHeader_1x02_P2.54mm_Vertical" H 950 3800 50  0001 C CNN
-F 3 "" H 950 3800 50  0001 C CNN
-	1    950  3800
+P 750 3700
+F 0 "SW1" V 796 3570 50  0000 R CNN
+F 1 "RESET" V 705 3570 50  0000 R CNN
+F 2 "8085:Switch_Tactile_SMD_6x6mm_PTS645" H 750 3700 50  0001 C CNN
+F 3 "" H 750 3700 50  0001 C CNN
+	1    750  3700
 	0    -1   -1   0
 $EndComp
@@
 L power:GND #PWR017
 U 1 1 5B8C4C86
-P 950 4150
-F 0 "#PWR017" H 950 3900 50  0001 C CNN
-F 1 "GND" H 955 3977 50  0000 C CNN
-F 2 "" H 950 4150 50  0001 C CNN
-F 3 "" H 950 4150 50  0001 C CNN
-	1    950  4150
-	1    0    0    -1
-$EndComp
-$Comp
-L Device:CP1 C8
-U 1 1 5B8C4CF6
-P 1450 3800
-F 0 "C8" H 1565 3846 50  0000 L CNN
-F 1 "1uF" H 1565 3755 50  0000 L CNN
-F 2 "Capacitor_THT:CP_Radial_D5.0mm_P2.50mm" H 1450 3800 50  0001 C CNN
-F 3 "~" H 1450 3800 50  0001 C CNN
-	1    1450 3800
-	1    0    0    -1
-$EndComp
-Wire Wire Line
-	1450 3650 1450 3500
-Connection ~ 1450 3500
-Wire Wire Line
-	950  3200 1450 3200
-Wire Wire Line
-	1450 4100 950  4100
-Wire Wire Line
-	1450 3950 1450 4100
-Wire Wire Line
-	950  4150 950  4100
-Connection ~ 950  4100
+P 750 4050
+F 0 "#PWR017" H 750 3800 50  0001 C CNN
+F 1 "GND" H 755 3877 50  0000 C CNN
+F 2 "" H 750 4050 50  0001 C CNN
+F 3 "" H 750 4050 50  0001 C CNN
+	1    750  4050
+	1    0    0    -1
+$EndComp
+Wire Wire Line
+	750  4050 750  4000
+Connection ~ 750  4000
 Wire Wire Line
 	6300 2200 6300 1550
@@
 Wire Wire Line
 	3500 3500 3500 3300
-Wire Wire Line
-	1450 3500 3500 3500
 Wire Wire Line
 	3250 3300 2250 3300
@@
 Wire Wire Line
 	4900 3400 9500 3400
-Text HLabel 6850 4900 2    50   Output ~ 0
-RESET
 Wire Wire Line
 	4900 4400 6200 4400
@@
 Wire Wire Line
 	3250 1700 3250 2000
+Text HLabel 2250 3200 0    50   Input ~ 0
+SID
+Text HLabel 6850 4900 2    50   Output ~ 0
+RESET
+Wire Wire Line
+	4900 4900 6850 4900
+Wire Bus Line
+	5750 1250 5750 2700
+$Comp
+L 8085:MCP1319 U5
+U 1 1 5D756153
+P 1450 3400
+F 0 "U5" H 1200 3800 50  0000 C CNN
+F 1 "MCP1319T-46LE" H 1850 2950 50  0000 C CNN
+F 2 "Package_TO_SOT_SMD:SOT-23-5_HandSoldering" H 1500 3400 50  0001 C CNN
+F 3 "" H 1500 3400 50  0001 C CNN
+	1    1450 3400
+	1    0    0    -1
+$EndComp
+Wire Wire Line
+	3500 3500 1800 3500
+NoConn ~ 1800 3300
+Wire Wire Line
+	1450 4000 1450 3850
+Wire Wire Line
+	750  4000 1450 4000
+Wire Wire Line
+	750  3400 1050 3400
+$Comp
+L power:VCC #PWR01
+U 1 1 5D76B360
+P 1450 2950
+F 0 "#PWR01" H 1450 2800 50  0001 C CNN
+F 1 "VCC" H 1467 3123 50  0000 C CNN
+F 2 "" H 1450 2950 50  0001 C CNN
+F 3 "" H 1450 2950 50  0001 C CNN
+	1    1450 2950
+	1    0    0    -1
+$EndComp
 Wire Wire Line
 	4900 2800 6900 2800
@@
 	4900 2100 6200 2100
 Wire Bus Line
-	5750 1250 5750 2700
+	9600 1500 9600 3500
 Wire Bus Line
 	8900 1300 8900 2250
-Wire Bus Line
-	9600 1500 9600 3500
 $EndSCHEMATC
