File: CPU8085.sch (KiCad schematic (older format))
At the start: 13 parts, among them J1 POWER, U1 GLUE_LOGIC

Commit message: RevB
Parts:
- removed J1: POWER, Connector_Molex:Molex_KK-254_AE-6410-04A_1x04_P2.54mm_Vertical, symbol Connector_Generic:Conn_01x04
- C1, C2, C3, C4, C5, C6, C7: footprint Capacitor_THT:C_Disc_D3.0mm_W2.0mm_P2.50mm -> Capacitor_SMD:C_0805_2012Metric_Pad1.15x1.40mm_HandSolder
Connections:
- wire segments 96 -> 88
Other:
- note added: "*POWER now comes from USB, see UART sheet"
Changed lines of the file:
@@
 EESchema Schematic File Version 4
-LIBS:CPU8085-cache
-EELAYER 26 0
+EELAYER 30 0
 EELAYER END
 $Descr USLetter 11000 8500
@@
 F7 "~RAMCE" I L 5800 5400 50
 $EndSheet
-$Comp
-L Connector_Generic:Conn_01x04 J1
-U 1 1 5B8BFF37
-P 900 1200
-F 0 "J1" H 820 1517 50  0000 C CNN
-F 1 "POWER" H 820 1426 50  0000 C CNN
-F 2 "Connector_Molex:Molex_KK-254_AE-6410-04A_1x04_P2.54mm_Vertical" H 900 1200 50  0001 C CNN
-F 3 "~" H 900 1200 50  0001 C CNN
-	1    900  1200
-	-1   0    0    -1
-$EndComp
-$Comp
-L power:GND #PWR02
-U 1 1 5B8C006F
-P 1250 1400
-F 0 "#PWR02" H 1250 1150 50  0001 C CNN
-F 1 "GND" H 1255 1227 50  0000 C CNN
-F 2 "" H 1250 1400 50  0001 C CNN
-F 3 "" H 1250 1400 50  0001 C CNN
-	1    1250 1400
-	1    0    0    -1
-$EndComp
-Wire Wire Line
-	1100 1300 1250 1300
-Wire Wire Line
-	1250 1300 1250 1400
-Wire Wire Line
-	1100 1400 1250 1400
-Connection ~ 1250 1400
-$Comp
-L power:VCC #PWR01
-U 1 1 5B8C00B4
-P 1250 1100
-F 0 "#PWR01" H 1250 950 50  0001 C CNN
-F 1 "VCC" H 1267 1273 50  0000 C CNN
-F 2 "" H 1250 1100 50  0001 C CNN
-F 3 "" H 1250 1100 50  0001 C CNN
-	1    1250 1100
-	1    0    0    -1
-$EndComp
-Wire Wire Line
-	1100 1100 1250 1100
-Wire Wire Line
-	1100 1200 1250 1200
-Wire Wire Line
-	1250 1200 1250 1100
-Connection ~ 1250 1100
-$Comp
-L power:PWR_FLAG #FLG01
-U 1 1 5B8D8E8F
-P 1550 1200
-F 0 "#FLG01" H 1550 1275 50  0001 C CNN
-F 1 "PWR_FLAG" V 1550 1328 50  0000 L CNN
-F 2 "" H 1550 1200 50  0001 C CNN
-F 3 "~" H 1550 1200 50  0001 C CNN
-	1    1550 1200
-	0    1    1    0
-$EndComp
-$Comp
-L power:PWR_FLAG #FLG02
-U 1 1 5B8D8EC7
-P 1550 1300
-F 0 "#FLG02" H 1550 1375 50  0001 C CNN
-F 1 "PWR_FLAG" V 1550 1428 50  0000 L CNN
-F 2 "" H 1550 1300 50  0001 C CNN
-F 3 "~" H 1550 1300 50  0001 C CNN
-	1    1550 1300
-	0    1    1    0
-$EndComp
-Connection ~ 1250 1200
-Connection ~ 1250 1300
 $Sheet
 S 5950 2600 1550 1500
@@
 F 0 "C1" H 8215 1496 50  0000 L CNN
 F 1 "0.1uF" H 8215 1405 50  0000 L CNN
-F 2 "Capacitor_THT:C_Disc_D3.0mm_W2.0mm_P2.50mm" H 8138 1300 50  0001 C CNN
+F 2 "Capacitor_SMD:C_0805_2012Metric_Pad1.15x1.40mm_HandSolder" H 8138 1300 50  0001 C CNN
 F 3 "~" H 8100 1450 50  0001 C CNN
 	1    8100 1450
@@
 F 0 "C2" H 8565 1496 50  0000 L CNN
 F 1 "0.1uF" H 8565 1405 50  0000 L CNN
-F 2 "Capacitor_THT:C_Disc_D3.0mm_W2.0mm_P2.50mm" H 8488 1300 50  0001 C CNN
+F 2 "Capacitor_SMD:C_0805_2012Metric_Pad1.15x1.40mm_HandSolder" H 8488 1300 50  0001 C CNN
 F 3 "~" H 8450 1450 50  0001 C CNN
 	1    8450 1450
@@
 F 0 "C3" H 8865 1496 50  0000 L CNN
 F 1 "0.1uF" H 8865 1405 50  0000 L CNN
-F 2 "Capacitor_THT:C_Disc_D3.0mm_W2.0mm_P2.50mm" H 8788 1300 50  0001 C CNN
+F 2 "Capacitor_SMD:C_0805_2012Metric_Pad1.15x1.40mm_HandSolder" H 8788 1300 50  0001 C CNN
 F 3 "~" H 8750 1450 50  0001 C CNN
 	1    8750 1450
@@
 F 0 "C4" H 9165 1496 50  0000 L CNN
 F 1 "0.1uF" H 9165 1405 50  0000 L CNN
-F 2 "Capacitor_THT:C_Disc_D3.0mm_W2.0mm_P2.50mm" H 9088 1300 50  0001 C CNN
+F 2 "Capacitor_SMD:C_0805_2012Metric_Pad1.15x1.40mm_HandSolder" H 9088 1300 50  0001 C CNN
 F 3 "~" H 9050 1450 50  0001 C CNN
 	1    9050 1450
@@
 F 0 "C5" H 9465 1496 50  0000 L CNN
 F 1 "0.1uF" H 9465 1405 50  0000 L CNN
-F 2 "Capacitor_THT:C_Disc_D3.0mm_W2.0mm_P2.50mm" H 9388 1300 50  0001 C CNN
+F 2 "Capacitor_SMD:C_0805_2012Metric_Pad1.15x1.40mm_HandSolder" H 9388 1300 50  0001 C CNN
 F 3 "~" H 9350 1450 50  0001 C CNN
 	1    9350 1450
@@
 F 0 "C6" H 9765 1496 50  0000 L CNN
 F 1 "0.1uF" H 9765 1405 50  0000 L CNN
-F 2 "Capacitor_THT:C_Disc_D3.0mm_W2.0mm_P2.50mm" H 9688 1300 50  0001 C CNN
+F 2 "Capacitor_SMD:C_0805_2012Metric_Pad1.15x1.40mm_HandSolder" H 9688 1300 50  0001 C CNN
 F 3 "~" H 9650 1450 50  0001 C CNN
 	1    9650 1450
@@
 F 0 "C7" H 10065 1496 50  0000 L CNN
 F 1 "0.1uF" H 10065 1405 50  0000 L CNN
-F 2 "Capacitor_THT:C_Disc_D3.0mm_W2.0mm_P2.50mm" H 9988 1300 50  0001 C CNN
+F 2 "Capacitor_SMD:C_0805_2012Metric_Pad1.15x1.40mm_HandSolder" H 9988 1300 50  0001 C CNN
 F 3 "~" H 9950 1450 50  0001 C CNN
 	1    9950 1450
@@
 Wire Wire Line
 	8150 3100 8800 3100
-Wire Wire Line
-	1250 1200 1550 1200
-Wire Wire Line
-	1250 1300 1550 1300
+Text Notes 6600 900  0    100  ~ 20
+*POWER now comes from USB, see UART sheet
 Wire Bus Line
 	3400 4900 3400 6150

Commit message: RevC
Parts:
- removed U1: GLUE_LOGIC, Package_DIP:DIP-20_W7.62mm, symbol 8085:GLUE_LOGIC
- added J3: PS2 KBD, 8085:CUI_MD-60S, symbol MD-60S:MD-60S
- added U1: DTGLUE4, Package_DIP:DIP-20_W7.62mm, symbol 8085:DTGLUE4
Connections:
- net A13: now also U1.4 (A13)
- net A14: now also U1.3 (A14)
- net A15: now also U1.2 (A15)
- net CPU/IO~M: now also U1.1 (IO/~M)
- net CPU/~RD: now also U1.6 (~RD)
- net CPU/~WR: now also U1.5 (~WR)
- net GND: now also U1.10 (GND)
- net PIT/~PIT: now also U1.18 (~PIT)
- net VCC: now also U1.20 (VCC)
- new net Memory/BANKREG: U1.19 (BANKREG)
- new net Sound (SN76489)/~SOUND: U1.15 (~SOUND)
- new net UART (FT240XS)/UART_WR: U1.17 (UART_WR)
- new net UART (FT240XS)/~UART_RD: U1.16 (~UART_RD)
Changed lines of the file:
@@
 Sheet 1 6
 Title "8085 MAIN BOARD"
-Date "2018-09-17"
-Rev "A"
+Date "2018-09-27"
+Rev "C"
 Comp ""
 Comment1 ""
@@
 $EndDescr
 $Sheet
-S 5800 4500 1650 1600
+S 5900 4500 1650 1600
 U 5B8BFECF
 F0 "Memory" 50
 F1 "Memory.sch" 50
-F2 "~ROMCE" I L 5800 5300 50
-F3 "~RD" I L 5800 5550 50
-F4 "A[0..15]" I L 5800 4900 50
-F5 "D[0..7]" B L 5800 4750 50
-F6 "~WR" I L 5800 5650 50
-F7 "~RAMCE" I L 5800 5400 50
+F2 "~RD" I L 5900 5550 50
+F3 "A[0..15]" I L 5900 4900 50
+F4 "D[0..7]" B L 5900 4750 50
+F5 "~WR" I L 5900 5650 50
+F6 "IO~M" I L 5900 5250 50
+F7 "BANKREG" I L 5900 5800 50
 $EndSheet
 $Sheet
 S 5950 2600 1550 1500
 U 5B955671
-F0 "UART" 50
-F1 "UART.sch" 50
+F0 "UART (FT240XS)" 50
+F1 "FT240XS.sch" 50
 F2 "D[0..7]" B L 5950 3750 50
-F3 "A[0..15]" I L 5950 3900 50
-F4 "CLOCK" I L 5950 3000 50
-F5 "RESET" I L 5950 3150 50
-F6 "~RD" I L 5950 3300 50
-F7 "~WR" I L 5950 3450 50
-F8 "~UART" I L 5950 3600 50
-F9 "~UART_OUT1" O R 7500 2800 50
-F10 "~UART_OUT2" O R 7500 2950 50
-F11 "INTR" O R 7500 3100 50
+F3 "~UART_RD" I L 5950 3450 50
+F4 "UART_WR" I L 5950 3600 50
+F5 "~RXF" O R 7500 3100 50
 $EndSheet
-Wire Bus Line
-	5050 3900 5050 4900
-Wire Bus Line
-	5050 3900 5350 3900
-Connection ~ 5050 4900
-Wire Bus Line
-	5050 4900 5800 4900
+Connection ~ 5350 4900
+Wire Bus Line
+	5350 4900 5900 4900
 Wire Bus Line
 	5950 3750 5200 3750
 Wire Bus Line
-	4850 3750 4850 4750
-Wire Bus Line
-	3250 4750 4850 4750
-Connection ~ 4850 4750
-Wire Bus Line
-	4850 4750 5800 4750
-Wire Wire Line
-	5950 3450 5000 3450
+	5200 3750 5200 4750
+Wire Bus Line
+	3250 4750 5200 4750
+Connection ~ 5200 4750
+Wire Bus Line
+	5200 4750 5700 4750
 Wire Wire Line
 	1100 3450 1100 5350
@@
 	1300 4950 1300 3000
 Wire Wire Line
-	1300 3000 5050 3000
-Wire Wire Line
-	5950 3150 1350 3150
-Wire Wire Line
-	1350 3150 1350 4750
-Wire Wire Line
-	1350 4750 1450 4750
+	1300 3000 4700 3000
 $Sheet
-S 5950 1350 1300 1000
+S 5950 1350 1550 1050
 U 5B98C06B
 F0 "PIT" 50
@@
 F7 "~PIT" I L 5950 1400 50
 F8 "TI_CLK" O L 5950 2300 50
-F9 "SPKR_EN" I R 7250 1800 50
-F10 "SPKR_OUT" O R 7250 1900 50
 $EndSheet
 Wire Wire Line
@@
 Connection ~ 4950 3300
 Wire Wire Line
-	4950 3300 5950 3300
-Wire Wire Line
 	5950 2050 5000 2050
 Wire Wire Line
@@
 Wire Wire Line
 	5050 2200 5050 3000
-Connection ~ 5050 3000
-Wire Wire Line
-	5050 3000 5950 3000
 Wire Bus Line
 	5950 1700 5350 1700
-Wire Bus Line
-	5350 1700 5350 3900
-Connection ~ 5350 3900
-Wire Bus Line
-	5350 3900 5950 3900
 Wire Bus Line
 	5950 1500 5200 1500
@@
 	5200 1500 5200 3750
 Connection ~ 5200 3750
-Wire Bus Line
-	5200 3750 4850 3750
-Wire Wire Line
-	1200 3300 4950 3300
-Wire Wire Line
-	1100 3450 5000 3450
+Wire Wire Line
+	1200 3300 3500 3300
+Wire Wire Line
+	1100 3450 3550 3450
 $Comp
 L Device:C C1
@@
 	5950 2300 900  2300
 Wire Wire Line
-	900  2300 900  5600
-Wire Wire Line
-	900  5600 1450 5600
+	900  2300 900  6000
+Wire Wire Line
+	900  6000 1450 6000
 $Sheet
-S 1450 4550 1800 1600
+S 1450 4550 1800 2100
 U 5B8BFEAE
 F0 "CPU" 50
@@
 F12 "RST6_5" I L 1450 5900 50
 F13 "RST7_5" I L 1450 6000 50
+F14 "SID" I L 1450 6150 50
 $EndSheet
 Wire Wire Line
-	5800 5550 4950 5550
+	5900 5550 4950 5550
 Wire Wire Line
 	4950 5550 4950 3300
 Wire Wire Line
-	5800 5650 5000 5650
-Wire Wire Line
-	5000 5650 5000 3450
-$Comp
-L 8085:GLUE_LOGIC U?
-U 1 1 5BC84670
-P 4300 6000
-AR Path="/5B8BFEAE/5BC84670" Ref="U?"  Part="1"
-AR Path="/5BC84670" Ref="U1"  Part="1"
-F 0 "U1" H 4000 6600 50  0000 C CNN
-F 1 "GLUE_LOGIC" H 4150 5400 50  0000 C CNN
-F 2 "Package_DIP:DIP-20_W7.62mm" H 4000 5450 50  0001 C CNN
-F 3 "" H 4000 5450 50  0001 C CNN
-	1    4300 6000
-	1    0    0    -1
-$EndComp
-Wire Wire Line
-	4750 5950 5700 5950
-Wire Wire Line
-	5700 5950 5700 5400
-Wire Wire Line
-	5700 5400 5800 5400
-Wire Wire Line
-	5650 5850 5650 5300
-Wire Wire Line
-	5650 5300 5800 5300
-Wire Wire Line
-	4750 6200 5600 6200
-Wire Wire Line
-	5600 6200 5600 3600
+	5900 5650 5000 5650
+Wire Wire Line
+	5000 5650 5000 4400
+Wire Wire Line
+	5600 6050 5600 3600
 Wire Wire Line
 	5600 3600 5950 3600
 Wire Wire Line
-	4750 5850 5650 5850
-Wire Wire Line
-	7500 2800 7750 2800
-Wire Wire Line
-	7750 2800 7750 6350
-Wire Wire Line
-	7750 6350 5500 6350
-Wire Wire Line
-	5500 6350 5500 6800
-Wire Wire Line
-	5500 6800 3700 6800
-Wire Wire Line
-	3700 6800 3700 6400
-Wire Wire Line
-	3700 6400 3850 6400
-Wire Wire Line
-	3850 5550 3250 5550
+	3850 5550 3700 5550
 Entry Wire Line
-	3400 5950 3500 6050
-Wire Wire Line
-	4750 6100 5550 6100
-Wire Wire Line
-	5550 6100 5550 1400
+	3400 5900 3500 6000
+Wire Wire Line
+	5550 5950 5550 1400
 Wire Wire Line
 	5550 1400 5950 1400
 Wire Wire Line
-	4750 6400 5450 6400
-Wire Wire Line
-	5450 6400 5450 6300
-Wire Wire Line
-	5450 6300 7950 6300
-Wire Wire Line
-	7950 6300 7950 1800
-Wire Wire Line
-	7950 1800 7250 1800
-Wire Bus Line
-	3250 4900 3400 4900
-Connection ~ 3400 4900
-Wire Bus Line
-	3400 4900 5050 4900
-Wire Wire Line
-	3850 6050 3500 6050
-Text Label 3700 6050 2    50   ~ 0
+	3850 6000 3500 6000
+Text Label 3700 6000 2    50   ~ 0
 A15
 Text Label 4150 4900 2    50   ~ 0
 A[0..15]
 Entry Wire Line
-	3400 6050 3500 6150
+	3400 6000 3500 6100
 Entry Wire Line
-	3400 6150 3500 6250
-Wire Wire Line
-	3500 6150 3850 6150
-Wire Wire Line
-	3500 6250 3850 6250
-Text Label 3700 6150 2    50   ~ 0
+	3400 6100 3500 6200
+Wire Wire Line
+	3500 6100 3850 6100
+Wire Wire Line
+	3500 6200 3850 6200
+Text Label 3700 6100 2    50   ~ 0
 A14
-Text Label 3700 6250 2    50   ~ 0
+Text Label 3700 6200 2    50   ~ 0
 A13
 Wire Wire Line
-	7500 2950 7600 2950
-NoConn ~ 7600 2950
-Wire Wire Line
 	7500 3100 7600 3100
 Wire Wire Line
-	7600 3100 7600 6400
-Wire Wire Line
-	7600 6400 5600 6400
-Wire Wire Line
-	5600 6400 5600 6850
+	7600 3100 7600 6650
+Wire Wire Line
+	7600 6650 5600 6650
+Wire Wire Line
+	5600 6650 5600 6850
 Wire Wire Line
 	5600 6850 1000 6850
 Wire Wire Line
-	1000 6850 1000 5900
-Wire Wire Line
-	1000 5900 1450 5900
+	1000 6850 1000 6150
+Wire Wire Line
+	1000 6150 1450 6150
 Wire Wire Line
 	8100 1300 8450 1300
@@
 Connection ~ 9750 2300
 $Sheet
-S 8800 2900 1400 1100
+S 8250 4550 1400 1100
 U 5BD66E5D
-F0 "SPEAKER" 50
-F1 "SPEAKER.sch" 50
-F2 "SPKR_IN" I L 8800 3100 50
+F0 "Sound (SN76489)" 50
+F1 "SN76489.sch" 50
+F2 "~SOUND" I L 8250 5500 50
+F3 "CLOCK" I L 8250 4700 50
+F4 "D[0..7]" I L 8250 5050 50
+F5 "~WR" I L 8250 5250 50
 $EndSheet
-Wire Wire Line
-	3850 6500 3850 6950
-Wire Wire Line
-	3850 6950 5700 6950
-Wire Wire Line
-	5700 6950 5700 6450
-Wire Wire Line
-	5700 6450 8000 6450
-Wire Wire Line
-	8000 6450 8000 1900
-Wire Wire Line
-	8000 1900 7250 1900
-Wire Wire Line
-	4750 6500 8150 6500
-Wire Wire Line
-	8150 6500 8150 3100
-Wire Wire Line
-	8150 3100 8800 3100
 Text Notes 6600 900  0    100  ~ 20
 *POWER now comes from USB, see UART sheet
-Wire Bus Line
-	3400 4900 3400 6150
+Wire Wire Line
+	5900 5250 3700 5250
+Wire Wire Line
+	3700 5250 3700 5550
+Connection ~ 3700 5550
+Wire Wire Line
+	3700 5550 3250 5550
+$Comp
+L 8085:DTGLUE4 U1
+U 1 1 5BAE4D96
+P 4300 6000
+F 0 "U1" H 4000 6600 50  0000 C CNN
+F 1 "DTGLUE4" H 4500 6600 50  0000 C CNN
+F 2 "Package_DIP:DIP-20_W7.62mm" H 4000 5400 50  0001 C CNN
+F 3 "" H 4000 5400 50  0001 C CNN
+	1    4300 6000
+	1    0    0    -1
+$EndComp
+Wire Wire Line
+	5900 5800 5000 5800
+Wire Wire Line
+	5000 5800 5000 5750
+Wire Wire Line
+	5000 5750 4750 5750
+Wire Wire Line
+	5550 5950 4750 5950
+Wire Wire Line
+	4750 6050 5600 6050
+Wire Bus Line
+	5700 4750 5700 4300
+Wire Bus Line
+	5700 4300 7750 4300
+Wire Bus Line
+	7750 4300 7750 5050
+Wire Bus Line
+	7750 5050 8250 5050
+Connection ~ 5700 4750
+Wire Bus Line
+	5700 4750 5900 4750
+Wire Wire Line
+	5000 4400 7700 4400
+Wire Wire Line
+	7700 4400 7700 5250
+Wire Wire Line
+	7700 5250 8250 5250
+Connection ~ 5000 4400
+Wire Wire Line
+	5000 4400 5000 3450
+Wire Wire Line
+	8000 6250 8000 5500
+Wire Wire Line
+	8000 5500 8250 5500
+Wire Wire Line
+	4700 3000 4700 4250
+Wire Wire Line
+	4700 4250 7850 4250
+Wire Wire Line
+	7850 4250 7850 4700
+Wire Wire Line
+	7850 4700 8250 4700
+Connection ~ 4700 3000
+Wire Wire Line
+	4700 3000 5050 3000
+Wire Wire Line
+	3850 5750 3550 5750
+Wire Wire Line
+	3550 5750 3550 3450
+Connection ~ 3550 3450
+Wire Wire Line
+	3550 3450 5000 3450
+Wire Bus Line
+	5350 1700 5350 4900
+Wire Wire Line
+	4750 6250 8000 6250
+Wire Bus Line
+	3250 4900 3400 4900
+Connection ~ 3400 4900
+Wire Bus Line
+	3400 4900 5350 4900
+Wire Wire Line
+	3850 5850 3500 5850
+Wire Wire Line
+	3500 5850 3500 3300
+Connection ~ 3500 3300
+Wire Wire Line
+	3500 3300 4950 3300
+Wire Wire Line
+	4750 6150 5650 6150
+Wire Wire Line
+	5650 6150 5650 3450
+Wire Wire Line
+	5650 3450 5950 3450
+NoConn ~ 1450 4750
+$Comp
+L MD-60S:MD-60S J3
+U 1 1 5BC56B60
+P 2700 1150
+F 0 "J3" H 2930 1146 50  0000 L CNN
+F 1 "PS2 KBD" H 2930 1055 50  0000 L CNN
+F 2 "8085:CUI_MD-60S" H 2700 1150 50  0001 L BNN
+F 3 "Manufacturer recommendations" H 2700 1150 50  0001 L BNN
+F 4 "CUI Inc." H 2700 1150 50  0001 L BNN "Field4"
+F 5 "1.03" H 2700 1150 50  0001 L BNN "Field5"
+	1    2700 1150
+	1    0    0    -1
+$EndComp
+Wire Bus Line
+	3400 4900 3400 6100
 $EndSCHEMATC
